File: SaberCord_Copy.kicad_pcb (KiCad board)
At the start: 2 copper layers, 2 parts

Commit message: refine footprint and schema
Parts:
- removed REF**: POGO, Connector:Tag-Connect_TC2070-IDC-FP_2x07_P1.27mm_Vertical
- removed REF**: Incoming, Connector_USB:USB_C_Receptacle_GCT_USB4085
- added J1: Conn_02x07_Row_Letter_Last, CommaPogo_Library:2x7_Pogo_Male, F.Cu at (139.7, 83.8)
- added J2: Conn_02x12_Row_Letter_Last, CommaPogo_Library:GCT_USB4056-03-A_REVA2, F.Cu at (140.0, 94.0)
Routing:
- net /GND: track 0.00 -> 33.4 mm
- net /CAN2_H: track 0.00 -> 19.3 mm
- net /CAN2_L: track 0.00 -> 18.5 mm
- net /VIN: track 0.00 -> 17.3 mm
- net /SBU2: track 0.00 -> 16.0 mm
- net /CAN3_H: track 0.00 -> 14.7 mm
- net /CAN0_H: track 0.00 -> 10.8 mm
- net /CAN3_L: track 0.00 -> 10.6 mm
- net /CAN0_L: track 0.00 -> 9.92 mm
- net /SBU1: track 0.00 -> 9.90 mm
- net /CAN1_H: track 0.00 -> 9.45 mm
- net /CAN1_L: track 0.00 -> 9.24 mm
Other:
- board outline added: 29.8 x 19.7 mm
