File: male_connector/SaberCord_Copy_Male.kicad_pcb (KiCad board)
At the start: 2 copper layers, 40.6 x 22.2 mm, 6 parts, among them J1 Conn_02x07_Row_Letter_Last, J2 Conn_02x12_Row_Letter_Last

Commit message: pcb finalized, very exciting
Routing:
- net GND: track 33.9 -> 48.8 mm
- net /CAN3_L: track 13.8 -> 16.8 mm
- net +12V: track 23.6 -> 25.0 mm
- net /CAN0_H: track 12.5 -> 13.5 mm
- net /SBU2: track 14.9 -> 15.0 mm, vias 0 -> 1
