File: female_connector/female_connector.kicad_sch (KiCad schematic)
At the start: 6 parts, among them J1 Conn_02x07_Row_Letter_Last, J2 Conn_02x12_Row_Letter_Last

Commit message: change usb c connector export to jlcpcb
Parts:
- J2: footprint CommaPogo_Library:GCT_USB4056-03-A_REVA2 -> CommaPogo_Library:USB-C-SMD_HC005-1A1H1A103-0HR; LCSC (none) -> C2894904
Changed lines of the file:
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@@
       (effects (font (size 1.27 1.27)) hide)
     )
-    (property "Footprint" "CommaPogo_Library:GCT_USB4056-03-A_REVA2" (at 166.37 95.25 0)
+    (property "Footprint" "CommaPogo_Library:USB-C-SMD_HC005-1A1H1A103-0HR" (at 166.37 95.25 0)
       (effects (font (size 1.27 1.27)) hide)
     )
@@
       (effects (font (size 1.27 1.27)) hide)
     )
+    (property "LCSC" "C2894904" (at 167.64 83.82 0)
+      (effects (font (size 1.27 1.27)) hide)
+    )
