File: commapogo_male/commapogo_male.kicad_sch (KiCad schematic)
At the start: 6 parts, among them J1 Conn_02x07_Row_Letter_Last, J2 Conn_02x12_Row_Letter_Last

Commit message: rework usb-c footprint for jlcpcb
Changed lines of the file:
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@@
   (paper "A4")
     (symbol "Connector_Generic:Conn_02x12_Row_Letter_Last" (pin_names (offset 1.016) hide) (in_bom yes) (on_board yes)
-      (property "Reference" "J2" (at 1.27 19.05 0)
+      (property "Reference" "J2" (at 1.27 16.51 0)
         (effects (font (size 1.27 1.27)))
       )
@@
         (effects (font (size 1.27 1.27)) hide)
       )
-      (property "Footprint" "Connector_USB:USB_C_Receptacle_CNCTech_C-ARA1-AK51X" (at 0 0 0)
+      (property "Footprint" "CommaPogo_Library:USB-C-SMD_HC005-1A1H1A103-0HR" (at 0 0 0)
         (effects (font (size 1.27 1.27)) hide)
       )
       (property "Datasheet" "~" (at 0 0 0)
+        (effects (font (size 1.27 1.27)) hide)
+      )
+      (property "LCSC" "C2894904" (at 1.27 11.43 0)
         (effects (font (size 1.27 1.27)) hide)
       )
@@
         )
         (pin passive line (at -5.08 12.7 0) (length 3.81)
-          (name "a1" (effects (font (size 1.27 1.27))))
+          (name "Pin_1a" (effects (font (size 1.27 1.27))))
           (number "A1" (effects (font (size 1.27 1.27))))
         )
         (pin passive line (at -5.08 -10.16 0) (length 3.81)
-          (name "a10" (effects (font (size 1.27 1.27))))
+          (name "Pin_10a" (effects (font (size 1.27 1.27))))
           (number "A10" (effects (font (size 1.27 1.27))))
         )
         (pin passive line (at -5.08 -12.7 0) (length 3.81)
-          (name "a11" (effects (font (size 1.27 1.27))))
+          (name "Pin_11a" (effects (font (size 1.27 1.27))))
           (number "A11" (effects (font (size 1.27 1.27))))
         )
         (pin passive line (at -5.08 -15.24 0) (length 3.81)
-          (name "a12" (effects (font (size 1.27 1.27))))
+          (name "Pin_12a" (effects (font (size 1.27 1.27))))
           (number "A12" (effects (font (size 1.27 1.27))))
         )
         (pin passive line (at -5.08 10.16 0) (length 3.81)
-          (name "a2" (effects (font (size 1.27 1.27))))
+          (name "Pin_2a" (effects (font (size 1.27 1.27))))
           (number "A2" (effects (font (size 1.27 1.27))))
         )
         (pin passive line (at -5.08 7.62 0) (length 3.81)
-          (name "a3" (effects (font (size 1.27 1.27))))
+          (name "Pin_3a" (effects (font (size 1.27 1.27))))
           (number "A3" (effects (font (size 1.27 1.27))))
         )
         (pin passive line (at -5.08 5.08 0) (length 3.81)
-          (name "a4" (effects (font (size 1.27 1.27))))
+          (name "Pin_4a" (effects (font (size 1.27 1.27))))
           (number "A4" (effects (font (size 1.27 1.27))))
         )
         (pin passive line (at -5.08 2.54 0) (length 3.81)
-          (name "a5" (effects (font (size 1.27 1.27))))
+          (name "Pin_5a" (effects (font (size 1.27 1.27))))
           (number "A5" (effects (font (size 1.27 1.27))))
         )
         (pin passive line (at -5.08 0 0) (length 3.81)
-          (name "a6" (effects (font (size 1.27 1.27))))
+          (name "Pin_6a" (effects (font (size 1.27 1.27))))
           (number "A6" (effects (font (size 1.27 1.27))))
         )
         (pin passive line (at -5.08 -2.54 0) (length 3.81)
-          (name "a7" (effects (font (size 1.27 1.27))))
+          (name "Pin_7a" (effects (font (size 1.27 1.27))))
           (number "A7" (effects (font (size 1.27 1.27))))
         )
         (pin passive line (at -5.08 -5.08 0) (length 3.81)
-          (name "A8" (effects (font (size 1.27 1.27))))
+          (name "Pin_8a" (effects (font (size 1.27 1.27))))
           (number "A8" (effects (font (size 1.27 1.27))))
         )
         (pin passive line (at -5.08 -7.62 0) (length 3.81)
-          (name "a9" (effects (font (size 1.27 1.27))))
+          (name "A9" (effects (font (size 1.27 1.27))))
           (number "A9" (effects (font (size 1.27 1.27))))
         )
         (pin passive line (at 7.62 12.7 180) (length 3.81)
-          (name "b1" (effects (font (size 1.27 1.27))))
+          (name "B1" (effects (font (size 1.27 1.27))))
           (number "B1" (effects (font (size 1.27 1.27))))
         )
         (pin passive line (at 7.62 -10.16 180) (length 3.81)
-          (name "b10" (effects (font (size 1.27 1.27))))
+          (name "Pin_10b" (effects (font (size 1.27 1.27))))
           (number "B10" (effects (font (size 1.27 1.27))))
         )
         (pin passive line (at 7.62 -12.7 180) (length 3.81)
-          (name "b11" (effects (font (size 1.27 1.27))))
+          (name "Pin_11b" (effects (font (size 1.27 1.27))))
           (number "B11" (effects (font (size 1.27 1.27))))
         )
         (pin passive line (at 7.62 -15.24 180) (length 3.81)
-          (name "b12" (effects (font (size 1.27 1.27))))
+          (name "Pin_12b" (effects (font (size 1.27 1.27))))
           (number "B12" (effects (font (size 1.27 1.27))))
         )
         (pin passive line (at 7.62 10.16 180) (length 3.81)
-          (name "b2" (effects (font (size 1.27 1.27))))
+          (name "Pin_2b" (effects (font (size 1.27 1.27))))
           (number "B2" (effects (font (size 1.27 1.27))))
         )
         (pin passive line (at 7.62 7.62 180) (length 3.81)
-          (name "b3" (effects (font (size 1.27 1.27))))
+          (name "Pin_3b" (effects (font (size 1.27 1.27))))
           (number "B3" (effects (font (size 1.27 1.27))))
         )
         (pin passive line (at 7.62 5.08 180) (length 3.81)
-          (name "b4" (effects (font (size 1.27 1.27))))
+          (name "Pin_4b" (effects (font (size 1.27 1.27))))
           (number "B4" (effects (font (size 1.27 1.27))))
         )
         (pin passive line (at 7.62 2.54 180) (length 3.81)
-          (name "b5" (effects (font (size 1.27 1.27))))
+          (name "Pin_5b" (effects (font (size 1.27 1.27))))
           (number "B5" (effects (font (size 1.27 1.27))))
         )
         (pin passive line (at 7.62 0 180) (length 3.81)
-          (name "b6" (effects (font (size 1.27 1.27))))
+          (name "Pin_6b" (effects (font (size 1.27 1.27))))
           (number "B6" (effects (font (size 1.27 1.27))))
         )
         (pin passive line (at 7.62 -2.54 180) (length 3.81)
-          (name "b7" (effects (font (size 1.27 1.27))))
+          (name "Pin_7b" (effects (font (size 1.27 1.27))))
           (number "B7" (effects (font (size 1.27 1.27))))
         )
         (pin passive line (at 7.62 -5.08 180) (length 3.81)
-          (name "b8" (effects (font (size 1.27 1.27))))
+          (name "Pin_8b" (effects (font (size 1.27 1.27))))
           (number "B8" (effects (font (size 1.27 1.27))))
         )
         (pin passive line (at 7.62 -7.62 180) (length 3.81)
-          (name "b9" (effects (font (size 1.27 1.27))))
+          (name "Pin_9b" (effects (font (size 1.27 1.27))))
           (number "B9" (effects (font (size 1.27 1.27))))
         )
@@
     (pin "9")
     (instances
-      (project "SaberCord_Copy_Male"
+      (project "commapogo_male"
         (path "/be2c8e72-e310-467f-9e4e-b384214483bd"
           (reference "J1") (unit 1)
@@
     )
     (instances
-      (project "SaberCord_Copy_Male"
+      (project "commapogo_male"
         (path "/be2c8e72-e310-467f-9e4e-b384214483bd"
           (reference "H4") (unit 1)
@@
     (pin "1")
     (instances
-      (project "SaberCord_Copy_Male"
+      (project "commapogo_male"
         (path "/be2c8e72-e310-467f-9e4e-b384214483bd"
           (reference "#PWR01") (unit 1)
@@
     (pin "1")
     (instances
-      (project "SaberCord_Copy_Male"
+      (project "commapogo_male"
         (path "/be2c8e72-e310-467f-9e4e-b384214483bd"
           (reference "#PWR02") (unit 1)
@@
     )
     (instances
-      (project "SaberCord_Copy_Male"
+      (project "commapogo_male"
         (path "/be2c8e72-e310-467f-9e4e-b384214483bd"
           (reference "H2") (unit 1)
@@
     )
     (instances
-      (project "SaberCord_Copy_Male"
+      (project "commapogo_male"
         (path "/be2c8e72-e310-467f-9e4e-b384214483bd"
           (reference "H3") (unit 1)
@@
     )
     (instances
-      (project "SaberCord_Copy_Male"
+      (project "commapogo_male"
         (path "/be2c8e72-e310-467f-9e4e-b384214483bd"
           (reference "H1") (unit 1)
@@
   )
   (symbol (lib_id "Connector_Generic:Conn_02x12_Row_Letter_Last") (at 166.37 95.25 0) (unit 1)
-    (in_bom yes) (on_board yes) (dnp no)
-    (property "Reference" "J2" (at 167.64 83.82 0)
+    (in_bom yes) (on_board yes) (dnp no) (fields_autoplaced)
+    (property "Reference" "J2" (at 167.64 78.74 0)
       (effects (font (size 1.27 1.27)))
     )
@@
       (effects (font (size 1.27 1.27)) hide)
     )
+    (pin "A10")
+    (pin "B10")
+    (pin "A11")
+    (pin "B11")
+    (pin "A12")
+    (pin "B12")
     (pin "A1")
-    (pin "A10")
-    (pin "A11")
-    (pin "A12")
+    (pin "B1")
     (pin "A2")
+    (pin "B2")
     (pin "A3")
+    (pin "B3")
     (pin "A4")
+    (pin "B4")
     (pin "A5")
+    (pin "B5")
     (pin "A6")
+    (pin "B6")
     (pin "A7")
+    (pin "B7")
     (pin "A8")
+    (pin "B8")
     (pin "A9")
-    (pin "B1")
-    (pin "B10")
-    (pin "B11")
-    (pin "B12")
-    (pin "B2")
-    (pin "B3")
-    (pin "B4")
-    (pin "B5")
-    (pin "B6")
-    (pin "B7")
-    (pin "B8")
     (pin "B9")
     (instances
-      (project "SaberCord_Copy_Male"
+      (project "commapogo_male"
         (path "/be2c8e72-e310-467f-9e4e-b384214483bd"
           (reference "J2") (unit 1)
