File: commapogo_male/commapogo_male.kicad_sch (KiCad schematic)
At the start: 6 parts, among them J1 Conn_02x07_Row_Letter_Last, J2 Conn_02x12_Row_Letter_Last

Commit message: revamp pcb design
Parts:
- H1, H2, H3, H4: footprint MountingHole:MountingHole_3mm -> MountingHole:MountingHole_2.2mm_M2
- J2: footprint CommaPogo_Library:USB-C-SMD_HC005-1A1H1A103-0HR -> CommaPogo_Library:GT-USB-7001C
Changed lines of the file:
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@@
 			)
 		)
-		(property "Footprint" "MountingHole:MountingHole_3mm"
+		(property "Footprint" "MountingHole:MountingHole_2.2mm_M2"
 			(at 134.62 135.89 0)
 			(effects
@@
 			)
 		)
-		(property "Footprint" "MountingHole:MountingHole_3mm"
+		(property "Footprint" "MountingHole:MountingHole_2.2mm_M2"
 			(at 118.11 135.89 0)
 			(effects
@@
 			)
 		)
-		(property "Footprint" "MountingHole:MountingHole_3mm"
+		(property "Footprint" "MountingHole:MountingHole_2.2mm_M2"
 			(at 134.62 128.27 0)
 			(effects
@@
 			)
 		)
-		(property "Footprint" "MountingHole:MountingHole_3mm"
+		(property "Footprint" "MountingHole:MountingHole_2.2mm_M2"
 			(at 118.11 128.27 0)
 			(effects
@@
 			)
 		)
-		(property "Footprint" "CommaPogo_Library:USB-C-SMD_HC005-1A1H1A103-0HR"
+		(property "Footprint" "CommaPogo_Library:GT-USB-7001C"
 			(at 166.37 95.25 0)
 			(effects
